Commit message: Updating husky_description.

File: husky_description/urdf/decorations.urdf.xacro (robot description, xacro)
@@ -22,5 +22,5 @@
     <!-- Attach chassis to the robot -->
     <joint name="top_chassis_joint" type="fixed">
-      <parent link="base_link" />
+      <parent link="${prefix}base_link" />
       <child link="top_chassis_link" />
     </joint>
@@ -37,5 +37,5 @@
       <joint name="user_rail" type="fixed">
         <origin xyz="0.272 0 0.245" rpy="0 0 0" />
-        <parent link="base_link" />
+        <parent link="${prefix}base_link" />
         <child link="user_rail_link" />
       </joint>
@@ -52,5 +52,5 @@
     <joint name="front_bumper" type="fixed">
       <origin xyz="${0.48 + husky_front_bumper_extend} 0 0.091" rpy="0 0 0" />
-      <parent link="base_link" />
+      <parent link="${prefix}base_link" />
       <child link="front_bumper_link" />
     </joint>
@@ -65,5 +65,5 @@
       <joint name="front_bumper_extension" type="fixed">
         <origin xyz="${0.48 + husky_front_bumper_extend} 0 0.091" rpy="0 0 0" />
-        <parent link="base_link" />
+        <parent link="${prefix}base_link" />
         <child link="front_bumper_extension_link" />
       </joint>
@@ -80,5 +80,5 @@
     <joint name="rear_bumper" type="fixed">
       <origin xyz="${-0.48 - husky_rear_bumper_extend} 0 0.091" rpy="0 0 ${M_PI}" />
-      <parent link="base_link" />
+      <parent link="${prefix}base_link" />
       <child link="rear_bumper_link" />
     </joint>
@@ -93,5 +93,5 @@
       <joint name="rear_bumper_extension" type="fixed">
         <origin xyz="${-0.48 - husky_rear_bumper_extend} 0 0.091" rpy="0 0 ${M_PI}" />
-        <parent link="base_link" />
+        <parent link="${prefix}base_link" />
         <child link="rear_bumper_extension_link" />
       </joint>
@@ -116,5 +116,5 @@
         <!-- Attach top plate -->
         <joint name="top_plate_joint" type="fixed">
-          <parent link="base_link" />
+          <parent link="${prefix}base_link" />
           <child link="top_plate_link"/>
           <origin xyz="0.0812 0 0.225" rpy="0 0 0"/>
@@ -150,5 +150,5 @@
         <!-- Attach top plate -->
         <joint name="top_plate_joint" type="fixed">
-          <parent link="base_link" />
+          <parent link="${prefix}base_link" />
           <child link="top_plate_link"/>
           <origin xyz="0.0812 0 0.245" rpy="0 0 0"/>

File: husky_description/urdf/husky_macro.urdf.xacro (robot description, xacro)
@@ -11,5 +11,6 @@
   <xacro:property name="husky_rear_bumper_extend" value="$(optenv HUSKY_REAR_BUMPER_EXTEND 0)" />
   <xacro:arg name="robot_namespace" default="/" />
-  <xacro:arg name="is_sim" default="false" />
+  <xacro:arg name="is_sim" default="true" />
+  <xacro:arg name="is_gazebo" default="false" />
   <xacro:arg name="urdf_extras" default="$(optenv CPR_URDF_EXTRAS empty.urdf)" />
   <!-- Included URDF/XACRO Files -->
@@ -135,6 +136,9 @@
     <ros2_control name="${prefix}husky_hardware" type="system">
       <hardware>
+        <xacro:if value="$(arg is_gazebo)">
+          <plugin>gazebo_ros2_control/GazeboSystem</plugin>
+        </xacro:if>
         <xacro:if value="$(arg is_sim)">
-          <plugin>gazebo_ros2_control/GazeboSystem</plugin>
+          <plugin>fake_components/GenericSystem</plugin>
         </xacro:if>
         <xacro:unless value="$(arg is_sim)">

File: husky_description/urdf/wheel.urdf.xacro (robot description, xacro)
@@ -1,5 +1,5 @@
 <?xml version="1.0"?>
 <robot xmlns:xacro="http://ros.org/wiki/xacro" name="husky_wheel">
-  <xacro:macro name="husky_wheel" params="wheel_prefix *joint_pose">
+  <xacro:macro name="husky_wheel" params="prefix wheel_prefix *joint_pose">
     <link name="${wheel_prefix}_wheel">
       <inertial>
@@ -29,5 +29,5 @@
     </gazebo>
     <joint name="${wheel_prefix}_wheel_joint" type="continuous">
-      <parent link="base_link"/>
+      <parent link="${prefix}base_link"/>
       <child link="${wheel_prefix}_wheel"/>
       <xacro:insert_block name="joint_pose"/>

Commit message: Fixing prefix parameter.

File: husky_description/urdf/decorations.urdf.xacro (robot description, xacro)
@@ -8,5 +8,5 @@
   <material name="white"><color rgba="1.0 1.0 1.0 1.0" /></material>
   <material name="red"><color rgba="1.0 0.0 0.0 1.0" /></material>
-  <xacro:macro name="husky_decorate">
+  <xacro:macro name="husky_decorate" params="prefix">
     <xacro:property name="husky_front_bumper_extend" value="$(optenv HUSKY_FRONT_BUMPER_EXTEND 0)" />
     <xacro:property name="husky_rear_bumper_extend" value="$(optenv HUSKY_REAR_BUMPER_EXTEND 0)" />

File: husky_description/urdf/husky_macro.urdf.xacro (robot description, xacro)
@@ -91,17 +91,17 @@
     </joint>
     <!-- Husky wheel macros -->
-    <xacro:husky_wheel wheel_prefix="${prefix}front_left">
+    <xacro:husky_wheel prefix="${prefix}" wheel_prefix="${prefix}front_left">
       <origin xyz="${wheelbase/2} ${track/2} ${wheel_vertical_offset}" rpy="0 0 0" />
     </xacro:husky_wheel>
-    <xacro:husky_wheel wheel_prefix="${prefix}front_right">
+    <xacro:husky_wheel prefix="${prefix}" wheel_prefix="${prefix}front_right">
       <origin xyz="${wheelbase/2} ${-track/2} ${wheel_vertical_offset}" rpy="0 0 0" />
     </xacro:husky_wheel>
-    <xacro:husky_wheel wheel_prefix="${prefix}rear_left">
+    <xacro:husky_wheel prefix="${prefix}" wheel_prefix="${prefix}rear_left">
       <origin xyz="${-wheelbase/2} ${track/2} ${wheel_vertical_offset}" rpy="0 0 0" />
     </xacro:husky_wheel>
-    <xacro:husky_wheel wheel_prefix="${prefix}rear_right">
+    <xacro:husky_wheel prefix="${prefix}" wheel_prefix="${prefix}rear_right">
       <origin xyz="${-wheelbase/2} ${-track/2} ${wheel_vertical_offset}" rpy="0 0 0" />
     </xacro:husky_wheel>
-    <xacro:husky_decorate />
+    <xacro:husky_decorate prefix="${prefix}" />
     <!-- <xacro:if value="$(arg laser_enabled)">
       <xacro:sick_lms1xx_mount prefix="base"/>
